File: pcb/mobo/mobo.kicad_pcb (KiCad board)
At the start: 2 copper layers, 51.6 x 89 mm, 72 parts, among them J1 SWD_10, J2 PEEL_MOTOR, J3 DRIVE_MOTOR, J4 SW1, J5 SPRING_FINGERS, J6 SW2, J7 SW1, J8 USART1, J9 SWD_10, U1 STM32F031C6Tx, U2 STM32F031K6Ux, U4 AP1117-33, U5 MC34063AD, U6 MAX3078E, U7 DRV8837, U8 DRV8837, Y1 8MHz

Commit message: Change 470uF electrolytic from 6.3mm to 8mm so there are more options available; Add LCSC, Mouser, and DigiKey reference parts.
Parts:
- removed the G*** at (107.0, 61.5)
- removed the G*** at (107.7, 98.4)
- removed REF**: OSHW-Symbol_6.7x6mm_Mask, feeder:OSHW-Symbol_6.7x6mm_Mask
- C1, C2: value 15p -> 15pF
- C16: footprint Capacitor_SMD:C_Elec_6.3x7.7 -> Capacitor_SMD:C_Elec_8x6.2
- J9: footprint feeder:SWD-No-Paste -> Connector_PinHeader_1.27mm:PinHeader_2x05_P1.27mm_Vertical_SMD
- U2: footprint feeder:QFN-32-No-Paste -> Package_DFN_QFN:QFN-32-1EP_5x5mm_P0.5mm_EP3.45x3.45mm
- moved D6 10.8 mm to (124.8, 41.5), turned to 90 degrees
- moved C6 4.78 mm to (115.0, 43.7)
- moved D2 3.03 mm to (112.2, 42.6), turned to 90 degrees
- moved R14 2.71 mm to (114.2, 46.5), turned to 180 degrees
- moved R9 2.46 mm to (118.3, 38.9)
- moved C14 2.32 mm to (121.8, 39.5), turned to 0 degrees
- moved R6 2.22 mm to (116.2, 38.9)
- moved C9 1.79 mm to (121.1, 51.4)
- moved C13 1.60 mm to (117.7, 51.4)
- moved D9 1.54 mm to (114.1, 50.0), turned to -90 degrees
- moved U4 1.34 mm to (119.7, 45.8)
- moved L1 1.30 mm to (126.9, 48.7)
- moved U5 1.05 mm to (128.8, 40.0)
- moved C16 0.92 mm to (134.8, 48.3)
- moved R13 0.66 mm to (124.3, 37.2)
Connections:
- D2 pad 1: RS-485- -> RS-485+
- D2 pad 2: RS-485+ -> RS-485-
Routing:
- net +3V3: track 269.4 -> 257.7 mm
- net SW2: track 55.1 -> 48.9 mm, vias 3 -> 2
- net RS-485-: track 16.4 -> 10.3 mm
- net RS-485+: track 15.5 -> 9.55 mm
- net Net-(J5-Pin_5): track 12.6 -> 9.45 mm
- net GND: track 39.6 -> 42.7 mm, vias 110 -> 122
- net SWCLK: track 50.8 -> 47.9 mm
- net 1WIRE: track 36.6 -> 39.2 mm
- net Net-(D6-K): track 10.0 -> 7.82 mm
- net SWDIO: track 52.5 -> 50.4 mm
- net Net-(U5-Vfb): track 14.5 -> 16.2 mm
- net Net-(U5-DC): track 9.45 -> 8.52 mm
- net +VDC: track 29.8 -> 28.9 mm
- net +10V: track 86.7 -> 85.9 mm
