File: pcb/mobo/mobo.kicad_sch (KiCad schematic)
At the start: 66 parts, among them J1 SWD_10, J2 PEEL_MOTOR, J3 DRIVE_MOTOR, J4 SW1, J5 SPRING_FINGERS, J6 SW2, J7 SW1, J8 USART1, J9 SWD_10, U1 STM32F031C6Tx, U2 STM32F031K6Ux, U4 AP1117-33, U5 MC34063AD, U6 MAX3078E, U7 DRV8837, U8 DRV8837, Y1 8MHz

Commit message: Change 470uF electrolytic from 6.3mm to 8mm so there are more options available; Add LCSC, Mouser, and DigiKey reference parts.
Parts:
- C1, C2: value 15p -> 15pF; DigiKey (none) -> 311-4165-1-ND; JLCPCB C1794 -> (none); LCSC C376865 -> C527077; Mouser (none) -> 603-CC805FRNPO9BN150; Notes (none) -> WARNING: old LCSC C476766 is 100nf cap
- C10, C11, C8: DigiKey (none) -> 1276-1248-1-ND; JLCPCB C49678 -> (none); LCSC C476766 -> C1779; Mouser (none) -> 187-CL21A475KBQNNNE; Notes (none) -> WARNING: old LCSC C476766 is 100nf cap
- C12: DigiKey (none) -> 565-EMZR500ARA101MF80GCT-ND; LCSC (none) -> C962164; Mouser (none) -> 661-EMZR500ARA101MF8
- C13, C9: DigiKey (none) -> 1276-1052-1-ND; JLCPCB C15850 -> (none); LCSC C17024 -> C15850; Mouser (none) -> 187-CL21A106KPFNNNE
- C14: DigiKey (none) -> 311-1124-1-ND; JLCPCB C49678 -> (none); LCSC C476766 -> C1743; Mouser (none) -> 603-CC805KRX7R9BB471; Notes (none) -> WARNING: LCSC C476766 is 100nf cap, Value is 470pf
- C16: footprint Capacitor_SMD:C_Elec_6.3x7.7 -> Capacitor_SMD:C_Elec_8x6.2; LCSC (none) -> C5354997; Notes (none) -> 6.3 or 8mm Diam, 7.7mm max Z-height; Previous was 6.3x7.7mm
- C17, C18, C19, C20, C3, C4, C5, C7: DigiKey (none) -> CL21B104KBCNNNL-ND; JLCPCB C49678 -> (none); Mouser (none) -> 187-CL21B104KBCNNNL; Notes (none) -> LCSCAlt: C913936
- C6: DigiKey (none) -> 311-4165-1-ND; JLCPCB C49678 -> (none); LCSC C476766 -> C527077; Mouser (none) -> 603-CC805FRNPO9BN150; Notes (none) -> WARNING: old LCSC C476766 is 100nf cap
- D1: DigiKey (none) -> 732-11414-1-ND; LCSC (none) -> C916078; Mouser (none) -> 710-155124M173200; Notes (none) -> WARNING: Footprints are close enough to LCSC one to work, n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
- D2: DigiKey (none) -> F6450CT-ND; Mouser (none) -> 576-SM712-02HTG; Notes (none) -> WARNING: old LCSC Part # didn't exist
- D3: LCSC (none) -> C458749; Mouser (none) -> 859-LTST-C19HE1WT
- D6: DigiKey (none) -> 1655-1N5819WCT-ND; LCSC (none) -> C963381; Mouser (none) -> 621-1N5819HW-F
- D9: DigiKey (none) -> MMSZ4684T1GOSCT-ND; JLCPCB MMSZ4684T1G -> (none); LCSC (none) -> C24672; Mouser (none) -> 863-MMSZ4684T1G
- FID1, FID2, FID3, J8, TP1, TP2, TP3, TP4, TP5, TP6, TP7, TP8: now not fitted
- J1, J9: Notes (none) -> WARNING: Is there room in the model for this; now not fitted
- J2, J3: DigiKey (none) -> WM1746-ND; Mouser (none) -> 538-53048-0610; Notes (none) -> MouserAlt: 53261-0671; DigiKeyAlt: WM7624CT-ND
- J5: DigiKey (none) -> 478-5453-1-ND; LCSC (none) -> C3035810; Mouser (none) -> 581-009155005541006
- L1: DigiKey (none) -> 535-13628-1-ND; LCSC C467145 -> C5127556; Mouser (none) -> 815-ASPIAIGS6055221T
- R1: DigiKey (none) -> YAG1240CT-ND; JLCPCB C17513 -> (none); Mouser (none) -> 603-RT0805FRE071KL
- R13: DigiKey (none) -> 13-RT0805FRE0733RLCT-ND; LCSC (none) -> C383899; Mouser (none) -> 603-RT0805FRE0733RL
- R14: DigiKey (none) -> 13-RT0805FRE07220RLCT-ND; LCSC (none) -> C17557; Mouser (none) -> 603-RT0805FRE07220RL
- R15, R16: DigiKey (none) -> 311-20.0CRCT-ND; LCSC (none) -> C17544; Mouser (none) -> 603-RC0805FR-0720RL
- R17, R4, R7: DigiKey (none) -> 311-10.0KCRCT-ND; JLCPCB C17513 -> (none); LCSC C17513 -> C84376; Mouser (none) -> 603-RC0805FR-0710KL; Notes (none) -> WARNING: Old LCSC C17513 part number is 1K resistor, value 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
- R2, R3, R5: DigiKey (none) -> 311-470ARCT-ND; JLCPCB C17710 -> (none); Mouser (none) -> 603-RC0805JR-07470RL
- R6: DigiKey (none) -> 311-5.60KCRCT-ND; LCSC (none) -> C4382; Mouser (none) -> 603-RC0805FR-075K6L
- R9: DigiKey (none) -> 311-39.0KCRCT-ND; LCSC (none) -> C113306; Mouser (none) -> 603-RC0805FR-0739KL
- U1: DigiKey (none) -> 497-13618-ND; LCSC (none) -> C329281; Mouser (none) -> 511-STM32F031C6T6; Notes (none) -> MouserAlt: 511-STM32F031C6T6TR
- U2: now left out of the parts list
- U4: DigiKey (none) -> AZ1117CH-3.3TRG1DICT-ND; JLCPCB C108785 -> (none); LCSC C92102 -> C5250992; Mouser (none) -> 621-AZ1117CH-3.3TRG1
- U5: DigiKey (none) -> 296-17765-1-ND; LCSC (none) -> C100023; Mouser (none) -> 595-MC34063ADR
- U6: DigiKey (none) -> MAX3078EESA+TCT-ND; JLCPCB C40031 -> (none); Mouser (none) -> 700-MAX3077EESAT
- U7, U8: DigiKey (none) -> 296-34806-1-ND; LCSC (none) -> C39159; Mouser (none) -> 595-DRV8837DSGR
- Y1: DigiKey (none) -> 50-ECS-80-18-33Q-CES-TRCT-ND; JLCPCB C253751 -> (none); LCSC C648984 -> C115962; Mouser (none) -> 520-80-18-33Q-CES-TR
Connections:
- net RS-485+: now also D2.1 (A1); no longer D2.2 (A2)
- net RS-485-: now also D2.2 (A2); no longer D2.1 (A1)
